Commit message: change collision box to pitch

File: resources/robots/b1z1/urdf/b1z1.urdf (robot description, URDF)
Before this commit: robot b1z1_description, 29 links, 28 joints
Links:
- link base: geometry visual box size=0.2 0.2 0.5

Commit message: Sample only stand
    - Sample using spherical coordinate with base quat
    - Shrink front legs when standing

File: resources/robots/b1z1/urdf/b1z1.urdf (robot description, URDF)
Before this commit: robot b1z1_description, 29 links, 28 joints
Links:
- link base: geometry visual box size=0.001 0.001 0.001
